File: Nostalgia.kicad_sch (KiCad schematic)
At the start: 26 parts, among them J10 490107670612, J20 USB-C6, U30 1117-3.3, U40 ESP32-S3-WROOM-1-N16R8

Commit message: Schemat
Parts:
- added BAT1, BAT2, BAT3: 18650, _custom:Bat_BH-18650-A1AJ005, symbol _custom:BATTERY
- added C1, C2: 10u, _custom:C_0603, symbol 000_moje:C
- added C3: 100n, _obudowy:C_0603, symbol 000_moje:C
- added C4, C5, C8, C9: 47uF 6.3V, _obudowy:C_0805, symbol 000_moje:C
- added C6, C7: 10u, _obudowy:C_0603, symbol 000_moje:C
- added D1, D2: LED, _custom:LED_0805, symbol _custom:LED
- added D3, D4: SS14, _obudowy:D_SMA_DO214AC, symbol 000_moje:SS14
- added K1, K10, K11, K12, K2, K3, K4, K5, K6, K7, K8, K9: TACT_6x3_SMD, _custom:TACT_6x3_SMD, symbol _custom:Z
- added K13, K14, K15, K16: TACT_6x6_SMD, _custom:TACT_6x6_SMD, symbol _custom:Z
- added L1, L3: 47uH, _obudowy:DLG-0504, symbol 000_moje:L
- added L2: 4.7uH, _obudowy:DLG-0504, symbol 000_moje:L
- added R1, R2: 1k, _custom:R_0603, symbol 000_moje:R
- added R3: 1k2, _custom:R_0603, symbol 000_moje:R
- added U1: TP4056, _custom:SO8-PowerPad, symbol 000_moje:TP4056
- added U2: TPS613222ADBV, _obudowy:SOT23-5, symbol 000_moje:TPS613222ADBV
- added U3: HT7750B-SOT23-3, _obudowy:SOT23, symbol 000_moje:HT7750B-SOT23-3
- added U4: HT7750B-SOT89, _obudowy:SOT89, symbol 000_moje:HT7750B-SOT89
- J20, R20, R21: now fitted
Connections:
- net 5V: no longer J20.A9 (VBUS), J20.B9 (VBUS)
- net GND: now also BAT1.2 (-), BAT2.2 (-), BAT3.2 (-), C1.2, C2.2, C3.2, C4.2, C5.2, C6.2, C7.2, C8.2, C9.2, R3.1, U1.1 (TEMP), U1.3 (GND), U1.9 (GND), U2.2 (GND), U3.1 (GND), U4.1 (GND)
- new net: R2.1, U1.7 (~{CHRG})
- new net: D2.1 (K), R2.2
- new net: D3.2 (A), L1.2, U3.3 (IN)
- new net: D4.2 (A), L3.2, U4.3 (IN)
- new net: L2.2, U2.1 (SW)
- new net: R3.2, U1.2 (PROG)
- new net: R1.1, U1.6 (~{STDBY})
- new net: D1.1 (K), R1.2
- new net 5VSW: C5.1, C6.1, C7.1, C9.1, D3.1 (K), D4.1 (K), U2.4 (OUT), U3.2 (OUT), U4.2 (OUT)
- new net VBAT: BAT1.1 (+), BAT2.1 (+), BAT3.1 (+), C1.1, U1.5 (BAT)
- new net VBATSW: C3.1, C4.1, C8.1, L1.1, L2.1, L3.1
- new net VUSB: C2.1, D1.2 (A), D2.2 (A), J20.A9 (VBUS), J20.B9 (VBUS), U1.4 (Vcc), U1.8 (CE)
Other:
- note added: "1000mA charging current"
- note added: "5V booster A - 0.5044 USD"
- note added: "5V booster B"
- note added: "5V booster C"
- note added: "Battery charger"
- note added: "Pobór prądu wyświetlacza: max 150mA"
- note added: "TPS63000 buck-boost"
- note added: "Ładowarka MCP73831"
- note removed: "USB Power"

Commit message: WIP
Parts:
- removed C3: 100n, _obudowy:C_0603, symbol 000_moje:C
- removed C4, C5, C8, C9: 47uF 6.3V, _obudowy:C_0805, symbol 000_moje:C
- removed C6, C7: 10u, _obudowy:C_0603, symbol 000_moje:C
- removed D3, D4: SS14, _obudowy:D_SMA_DO214AC, symbol 000_moje:SS14
- removed L1, L3: 47uH, _obudowy:DLG-0504, symbol 000_moje:L
- removed L2: 4.7uH, _obudowy:DLG-0504, symbol 000_moje:L
- removed U2: TPS613222ADBV, _obudowy:SOT23-5, symbol 000_moje:TPS613222ADBV
- removed U3: HT7750B-SOT23-3, _obudowy:SOT23, symbol 000_moje:HT7750B-SOT23-3
- removed U30: 1117-3.3, _custom:SOT223, symbol _custom:1117-X.X
- removed U4: HT7750B-SOT89, _obudowy:SOT89, symbol 000_moje:HT7750B-SOT89
- added C10, C4, C5: 10u, _custom:C_0603, symbol _custom:C
- added L4: 4.7uH, symbol _custom:L
- added U5: TPS613222ADBV, _custom:SOT23-5, symbol _custom:TPS613222ADBV
Connections:
- net 5V: now also C4.1, C5.1, U5.4 (OUT); no longer J10.2 (Pin_2)
- net GND: now also C10.2, C4.2, C5.2, U5.2 (GND)
- net VBAT: now also C10.1, L4.1
- net VUSB: now also J10.2 (Pin_2)
- new net: L4.2, U5.1 (SW)
Other:
- note removed: "5V booster A - 0.5044 USD"
- note removed: "5V booster B"
- note removed: "5V booster C"

Commit message: WIP
Parts:
- removed C30, C32: 10u, _custom:C_0603, symbol _custom:C
- removed C31, C33: 1u, _custom:C_0603, symbol _custom:C
- removed FID1, FID2, FID3, FID4, FID5, FID6: 1.00mm, _custom:Fiducial_1.00mm, symbol _custom:_FIDUCIAL
- added C3, C6, C8: 10u, _custom:C_0603, symbol _custom:C
- added C7: 100n, _custom:C_0603, symbol _custom:C
- added DISP1: OLED, _custom:OLED_2.42inch_board, symbol Connector_Generic:Conn_01x04
- added L1: 2.2uH, _custom:DJNR3015, symbol _custom:L
- added R4: 1M, _custom:R_0603, symbol 000_moje:R
- added R5: 180k, _custom:R_0603, symbol 000_moje:R
- added R6: 100R, _custom:R_0603, symbol 000_moje:R
- added U2: TPS63000, _custom:Texas_DRC0010J_ThermalVias, symbol _custom:TPS63000
- L4: footprint (none) -> _custom:DJNR3015
Connections:
- net 3V3: now also C6.1, C8.1, R4.2, U2.1 (VOUT)
- net 5V: now also DISP1.2 (Pin_2)
- net GND: now also C3.2, C6.2, C7.2, C8.2, DISP1.1 (Pin_1), R5.1, U2.11 (PAD), U2.3 (PGND), U2.9 (GND)
- net VBAT: now also C3.1, R6.2, U2.5 (VIN)
- new net: R4.1, R5.2, U2.10 (FB)
- new net: L1.2, U2.2 (L2)
- new net: L1.1, U2.4 (L1)
- new net: C7.1, R6.1, U2.6 (EN), U2.7 (PS), U2.8 (VINA)
- new net SCL: DISP1.3 (Pin_3)
- new net SDA: DISP1.4 (Pin_4)
Other:
- note added: "V_{FB}=500mV"
- note removed: "Power supply"
