File: Nostalgia.kicad_sch (KiCad schematic)
At the start: 57 parts, among them J10 490107670612, J20 USB-C6, K1 TACT_6x3_SMD, K10 TACT_6x3_SMD, K11 TACT_6x3_SMD, K12 TACT_6x3_SMD, K13 TACT_6x6_SMD, K14 TACT_6x6_SMD, K15 TACT_6x6_SMD, K16 TACT_6x6_SMD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

Commit message: WIP
Parts:
- added R7: 1M, _custom:R_0603, symbol 000_moje:R
Connections:
- net Col0: now also K1.1, K10.1, K4.1, K7.1
- net Col1: now also K11.1, K2.1, K5.1, K8.1
- net Col2: now also K12.1, K3.1, K6.1, K9.1
- net Col3: now also K13.1, K14.1, K15.1, K16.1
- net Row0: now also K1.2, K14.2, K2.2, K3.2
- net Row1: now also K15.2, K4.2, K5.2, K6.2
- net Row2: now also K13.2, K7.2, K8.2, K9.2
- net Row3: now also K10.2, K11.2, K12.2, K16.2
Other:
- moved on the sheet: K1, K10, K11, K12, K13, K14, K15, K16, K2, K3, K4, K5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

Commit message: WIP
Parts:
- added DISP2: OLED, _custom:OLED_2.42inch_board_2, symbol Connector_Generic:Conn_01x07
Changed lines of the file:
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@@
+	)
+	(symbol
+		(lib_id "Connector_Generic:Conn_01x07")
+		(at 120.65 140.97 0)
+		(unit 1)
+		(exclude_from_sim no)
+		(in_bom yes)
+		(on_board yes)
+		(dnp no)
+		(property "Reference" "DISP2"
+			(at 120.65 130.81 0)
+			(effects
+				(font
+					(size 1.27 1.27)
+				)
+			)
+		)
+		(property "Value" "OLED"
+			(at 120.65 151.13 0)
+			(effects
+				(font
+					(size 1.27 1.27)
+				)
+			)
+		)
+		(property "Footprint" "_custom:OLED_2.42inch_board_2"
+			(at 120.65 140.97 0)
+			(effects
+				(font
+					(size 1.27 1.27)
+				)
+				(hide yes)
+			)
+		)
+		(property "Datasheet" "~"
+			(at 120.65 140.97 0)
+			(effects
+				(font
+					(size 1.27 1.27)
+				)
+				(hide yes)
+			)
+		)
+		(property "Description" "Generic connector, single row, 01x07, script generated (kicad-library-utils/schlib/autogen/connector/)"
+			(at 120.65 140.97 0)
+			(effects
+				(font
+					(size 1.27 1.27)
+				)
+				(hide yes)
+			)
+		)
+		(pin "6"
+		)
+		(pin "3"
+		)
+		(pin "2"
+		)
+		(pin "7"
+		)
+		(pin "5"
+		)
+		(pin "1"
+		)
+		(pin "4"
+		)
+		(instances
+			(project ""
+				(path "/8c2261c3-2d54-4beb-9b6c-a4aaa148eb6b"
+					(reference "DISP2")
+					(unit 1)
+				)
+			)
+		)
 	)
 	(symbol

Commit message: Wydłużenie płytki i zmiana przycisków z 6x3 na 6x6
Parts:
- K1, K10, K11, K12, K2, K3, K4, K5, K6, K7, K8, K9: footprint _custom:TACT_6x3_SMD -> _custom:TACT_6x6_SMD
Changed lines of the file:
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@@
 			)
 		)
-		(property "Footprint" "_custom:TACT_6x3_SMD"
+		(property "Footprint" "_custom:TACT_6x6_SMD"
 			(at 223.52 36.83 0)
 			(effects
@@
 			)
 		)
-		(property "Footprint" "_custom:TACT_6x3_SMD"
+		(property "Footprint" "_custom:TACT_6x6_SMD"
 			(at 223.52 45.72 0)
 			(effects
@@
 			)
 		)
-		(property "Footprint" "_custom:TACT_6x3_SMD"
+		(property "Footprint" "_custom:TACT_6x6_SMD"
 			(at 236.22 63.5 0)
 			(effects
@@
 			)
 		)
-		(property "Footprint" "_custom:TACT_6x3_SMD"
+		(property "Footprint" "_custom:TACT_6x6_SMD"
 			(at 248.92 63.5 0)
 			(effects
@@
 			)
 		)
-		(property "Footprint" "_custom:TACT_6x3_SMD"
+		(property "Footprint" "_custom:TACT_6x6_SMD"
 			(at 223.52 63.5 0)
 			(effects
@@
 			)
 		)
-		(property "Footprint" "_custom:TACT_6x3_SMD"
+		(property "Footprint" "_custom:TACT_6x6_SMD"
 			(at 236.22 54.61 0)
 			(effects
@@
 			)
 		)
-		(property "Footprint" "_custom:TACT_6x3_SMD"
+		(property "Footprint" "_custom:TACT_6x6_SMD"
 			(at 223.52 54.61 0)
 			(effects
@@
 			)
 		)
-		(property "Footprint" "_custom:TACT_6x3_SMD"
+		(property "Footprint" "_custom:TACT_6x6_SMD"
 			(at 248.92 36.83 0)
 			(effects
@@
 			)
 		)
-		(property "Footprint" "_custom:TACT_6x3_SMD"
+		(property "Footprint" "_custom:TACT_6x6_SMD"
 			(at 236.22 36.83 0)
 			(effects
@@
 			)
 		)
-		(property "Footprint" "_custom:TACT_6x3_SMD"
+		(property "Footprint" "_custom:TACT_6x6_SMD"
 			(at 236.22 45.72 0)
 			(effects
@@
 			)
 		)
-		(property "Footprint" "_custom:TACT_6x3_SMD"
+		(property "Footprint" "_custom:TACT_6x6_SMD"
 			(at 248.92 54.61 0)
 			(effects
@@
 			)
 		)
-		(property "Footprint" "_custom:TACT_6x3_SMD"
+		(property "Footprint" "_custom:TACT_6x6_SMD"
 			(at 248.92 45.72 0)
 			(effects

Commit message: WIP
Parts:
- removed C10, C4, C5: 10u, _custom:C_0603, symbol _custom:C
- removed DISP1: OLED, _custom:OLED_2.42inch_board, symbol Connector_Generic:Conn_01x04
- removed L4: 4.7uH, _custom:DJNR3015, symbol _custom:L
- removed R7: 1M, _custom:R_0603, symbol 000_moje:R
- removed TP3: 5V, _custom:Testpoint_2.00mm, symbol _custom:TP
- removed U5: TPS613222ADBV, _custom:SOT23-5, symbol _custom:TPS613222ADBV
- added C22, C40: 100n, _custom:C_0805, symbol _custom:C
- added C41: 10u, _custom:C_0805, symbol _custom:C
- added PMOD1, PMOD2: Conn_02x06_Top_Bottom, _custom:PMOD, symbol Connector_Generic:Conn_02x06_Top_Bottom
- added R25, R26: xxx, _custom:R_0805, symbol 000_moje:R
- C10: renamed from C40; value 100n -> 1u; footprint _custom:C_0603 -> _custom:C_0805
- C11: renamed from C41; footprint _custom:C_0603 -> _custom:C_0805
- C12: renamed from C42; footprint _custom:C_0603 -> _custom:C_0805
- C13: renamed from C43; footprint _custom:C_0603 -> _custom:C_0805
- C14: renamed from C44; footprint _custom:C_0603 -> _custom:C_0805
- C20: renamed from C2; footprint _custom:C_0603 -> _custom:C_0805
- C21: renamed from C1; footprint _custom:C_0603 -> _custom:C_0805
- C30: renamed from C3; footprint _custom:C_0603 -> _custom:C_0805
- C31: renamed from C7; footprint _custom:C_0603 -> _custom:C_0805
- C32: renamed from C6; footprint _custom:C_0603 -> _custom:C_0805
- C33: renamed from C8; footprint _custom:C_0603 -> _custom:C_0805
- DISP1: renamed from DISP2; footprint _custom:OLED_2.42inch_board_2 -> _custom:OLED_2.42inch_board_3
- K1, K10, K11, K12, K2, K3, K4, K5, K6, K7, K8, K9: value TACT_6x3_SMD -> TACT_6x6_SMD
- R10: renamed from R40; footprint _custom:R_0603 -> _custom:R_0805
- R20, R21: footprint _custom:R_0603 -> _custom:R_0805
- R22: renamed from R1; footprint _custom:R_0603 -> _custom:R_0805
- R23: renamed from R2; footprint _custom:R_0603 -> _custom:R_0805
- R24: renamed from R3; footprint _custom:R_0603 -> _custom:R_0805
- R30: renamed from R6; footprint _custom:R_0603 -> _custom:R_0805
- R31: renamed from R4; footprint _custom:R_0603 -> _custom:R_0805
- R32: renamed from R5; footprint _custom:R_0603 -> _custom:R_0805
- renumbered L1 to L30, U40 to U10, U1 to U20, U2 to U30
Connections:
- net Col3 is gone; now on net GND: K13.1, K14.1, K15.1, K16.1
- net 3V3: now also C40.1, C41.1, PMOD1.12 (Pin_12), PMOD1.6 (Pin_6), PMOD2.12 (Pin_12), PMOD2.6 (Pin_6)
- net GND: now also C22.2, C40.2, C41.2, PMOD1.11 (Pin_11), PMOD1.5 (Pin_5), PMOD2.11 (Pin_11), PMOD2.5 (Pin_5), R26.1
- net Row0: no longer K14.2
- net Row1: no longer K15.2
- net Row2: no longer K13.2
- net Row3: no longer K16.2
- net VBAT: now also R25.2
- new net ADC-Bat: C22.1, R25.1, R26.2
- new net ButtonDown: K15.2
- new net ButtonLeft: K13.2
- new net ButtonRigth: K16.2
- new net ButtonUp: K14.2
Other:
- note added: "Buck-boost"
- note added: "Buttons"
- note added: "Display"
- note added: "Matrix Keyboard"
- note added: "RTC piny 0-21 Analog piny 1-20 ADC1 piny 1-10 ADC2 piny 11-20 (nie działa razem z wifi) ADC zakresy: 0...850mV ACD rozdzielczość 12-bit"
- note removed: "TPS63000 buck-boost"
- note removed: "https://www.lcsc.com/product-detail/Button-And-Strip-Battery-Connector_MYOUNG-BH-18650-A1AJ005_C5290176.html?s_z=n_18650"
- note removed: "Ładowarka MCP73831"
- moved on the sheet: BAT1, BAT2, BAT3, C20, C21, C30, C31, C32, C33, D1, D2, DISP1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

Commit message: WIP
Connections:
- net 3V3: now also DISP1.1 (Pin_1), DISP1.7 (Pin_7)
- net GND: now also DISP1.2 (Pin_2), DISP1.6 (Pin_6)
- net SCL: now also DISP1.5 (Pin_5)
- net SDA: now also DISP1.4 (Pin_4)
- no-connect marks 3 -> 4
Changed lines of the file:
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@@
 		(at 63.5 129.54)
 	)
+	(no_connect
+		(at 217.17 58.42)
+	)
 	(wire
 		(pts
@@
 	(wire
 		(pts
+			(xy 203.2 58.42) (xy 213.36 58.42)
+		)
+		(stroke
+			(width 0)
+			(type default)
+		)
+	)
+	(wire
+		(pts
 			(xy 139.7 64.77) (xy 139.7 69.85)
 		)
@@
 	(wire
 		(pts
+			(xy 209.55 60.96) (xy 217.17 60.96)
+		)
+		(stroke
+			(width 0)
+			(type default)
+		)
+	)
+	(wire
+		(pts
 			(xy 27.94 161.29) (xy 30.48 161.29)
 		)
@@
 	(wire
 		(pts
+			(xy 210.82 55.88) (xy 217.17 55.88)
+		)
+		(stroke
+			(width 0)
+			(type default)
+		)
+	)
+	(wire
+		(pts
 			(xy 123.19 139.7) (xy 123.19 140.97)
 		)
@@
 	(wire
 		(pts
+			(xy 209.55 63.5) (xy 217.17 63.5)
+		)
+		(stroke
+			(width 0)
+			(type default)
+		)
+	)
+	(wire
+		(pts
 			(xy 189.23 154.94) (xy 189.23 147.32)
 		)
@@
 	(wire
 		(pts
+			(xy 210.82 66.04) (xy 217.17 66.04)
+		)
+		(stroke
+			(width 0)
+			(type default)
+		)
+	)
+	(wire
+		(pts
 			(xy 196.85 147.32) (xy 204.47 147.32)
 		)
@@
 	(wire
 		(pts
+			(xy 210.82 68.58) (xy 217.17 68.58)
+		)
+		(stroke
+			(width 0)
+			(type default)
+		)
+	)
+	(wire
+		(pts
 			(xy 27.94 158.75) (xy 30.48 158.75)
 		)
@@
 		(pts
 			(xy 317.5 95.25) (xy 318.77 95.25)
+		)
+		(stroke
+			(width 0)
+			(type default)
+		)
+	)
+	(wire
+		(pts
+			(xy 210.82 53.34) (xy 217.17 53.34)
 		)
 		(stroke
@@
 		)
 	)
+	(label "DispReset"
+		(at 203.2 58.42 0)
+		(effects
+			(font
+				(size 1.27 1.27)
+			)
+			(justify left bottom)
+		)
+	)
 	(label "Row0"
 		(at 106.68 60.96 0)
@@
 		)
 	)
+	(label "3V3"
+		(at 210.82 53.34 0)
+		(effects
+			(font
+				(size 1.27 1.27)
+			)
+			(justify left bottom)
+		)
+	)
 	(label "SCL"
 		(at 77.47 158.75 180)
@@
 		)
 	)
+	(label "SCL"
+		(at 209.55 63.5 0)
+		(effects
+			(font
+				(size 1.27 1.27)
+			)
+			(justify left bottom)
+		)
+	)
 	(label "SDA"
 		(at 77.47 161.29 180)
@@
 		)
 	)
+	(label "GND"
+		(at 210.82 55.88 0)
+		(effects
+			(font
+				(size 1.27 1.27)
+			)
+			(justify left bottom)
+		)
+	)
 	(label "Row3"
 		(at 76.2 80.01 180)
@@
 		)
 	)
+	(label "SDA"
+		(at 209.55 60.96 0)
+		(effects
+			(font
+				(size 1.27 1.27)
+			)
+			(justify left bottom)
+		)
+	)
 	(label "ButtonUp"
 		(at 163.83 44.45 0)
@@
 		)
 	)
+	(label "3V3"
+		(at 210.82 68.58 0)
+		(effects
+			(font
+				(size 1.27 1.27)
+			)
+			(justify left bottom)
+		)
+	)
 	(label "Col2"
 		(at 76.2 87.63 180)
@@
 		(effects
 			(font
+				(size 1.27 1.27)
+			)
+			(justify left bottom)
+		)
+	)
+	(label "GND"
+		(at 210.82 66.04 0)
+		(effects
+			(font

Commit message: WIP
Other:
- note added: "INT"
- note added: "MISO Rx"
- note added: "MOSI Tx"
- note added: "RESET"
- note added: "SCK"
- note added: "SCL"
- note added: "SDA"
- note added: "SS"
- moved on the sheet: BAT1, BAT2, BAT3, C20, C21, C22, C30, C31, C32, C33, D1, D2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

Commit message: Schemat prawie gotowy
Parts:
- C20, C21: symbol 000_moje:C -> _custom:C
- L30: footprint _custom:DJNR3015 -> _custom:DJNR5050
- R22, R23, R24, R25, R26, R30, R31, R32: symbol 000_moje:R -> _custom:R
- U20: symbol 000_moje:TP4056 -> _custom:TP4056
Connections:
- net ADC-Bat: now also U10.39 (IO1)
- net ButtonDown: now also U10.5 (IO5)
- net ButtonLeft: now also U10.6 (IO6)
- net ButtonRigth: now also U10.7 (IO7)
- net ButtonUp: now also U10.4 (IO4)
- net Col0: now also U10.14 (D+/IO20)
- net Col1: now also U10.23 (IO21)
- net Col2: now also U10.31 (IO38)
- net Row0: now also U10.9 (XTAL/IO16)
- net Row1: now also U10.10 (Tx1/IO17)
- net Row2: now also U10.11 (Rx1/IO18)
- net Row3: now also U10.13 (D-/IO19)
- net SCL: now also U10.38 (IO2)
- net SDA: now also U10.15 (JTAG/IO3)
- net GPIO8: now reaches U10.12 (IO8)
- net GPIO8: now also PMOD1.10 (Pin_10)
- net GPIO46: now reaches U10.16 (Log/IO46)
- net GPIO46: now also PMOD2.8 (Pin_8)
- net GPIO9: now reaches U10.17 (IO9)
- net GPIO9: now also PMOD1.9 (Pin_9)
- net GPIO10: now reaches U10.18 (IO10)
- net GPIO10: now also PMOD1.1 (Pin_1)
- net GPIO11: now reaches U10.19 (IO11)
- net GPIO11: now also PMOD1.2 (Pin_2)
- net GPIO12: now reaches U10.20 (IO12)
- net GPIO12: now also PMOD1.4 (Pin_4)
- net GPIO13: now reaches U10.21 (IO13)
- net GPIO13: now also PMOD1.3 (Pin_3)
- net GPIO14: now reaches U10.22 (IO14)
- net GPIO14: now also PMOD1.8 (Pin_8)
- net GPIO47: now reaches U10.24 (IO47)
- net GPIO47: now also PMOD2.9 (Pin_9)
- net GPIO48: now reaches U10.25 (IO48)
- net GPIO48: now also PMOD2.10 (Pin_10)
- net GPIO45: now reaches U10.26 (MemVolt/IO45)
- net GPIO45: now also PMOD2.7 (Pin_7)
- net GPIO39: now reaches U10.32 (MTCK/IO39)
- net GPIO39: now also PMOD2.1 (Pin_1)
- net GPIO40: now reaches U10.33 (MTDO/IO40)
- net GPIO40: now also PMOD2.2 (Pin_2)
- net GPIO41: now reaches U10.34 (MTDI/IO41)
- net GPIO41: now also PMOD2.3 (Pin_3)
- net GPIO42: now reaches U10.35 (MTMS/IO42)
- net GPIO42: now also PMOD2.4 (Pin_4)
- net GPIO15: now reaches U10.8 (XTAL/IO15)
- net GPIO15: now also PMOD1.7 (Pin_7)
Other:
- note added: "I2C Address: 0x3C"
- note added: "PMOD1"
- note added: "RTC piny 0-21 Analog piny 1-20 ADC1 piny 1-10 ADC2 piny 11-20 (nie działa razem z wifi) ADC zakresy: 0...850mV ADC rozdzielczość 12-bit"
- note removed: "RTC piny 0-21 Analog piny 1-20 ADC1 piny 1-10 ADC2 piny 11-20 (nie działa razem z wifi) ADC zakresy: 0...850mV ACD rozdzielczość 12-bit"
- moved on the sheet: LOGO1

Commit message: Włącznik zasilania
Parts:
- added K17: YUEN_FUNG_ST-0-102-C03-N003-RS, _custom:YUEN_FUNG_ST-0-102-C03-N003-RS, symbol _custom:Z
Connections:
- net VBAT: now also K17.1; no longer BAT1.1 (+), BAT2.1 (+), BAT3.1 (+), C21.1, R25.2, U20.5 (BAT)
- new net: BAT1.1 (+), BAT2.1 (+), BAT3.1 (+), C21.1, K17.2, R25.2, U20.5 (BAT)
Other:
- moved on the sheet: C30, C31, C32, C33, L30, R30, R31, R32, U30
