File: Nostalgia.kicad_sch (KiCad schematic)
At the start: 59 parts, among them J10 490107670612, J20 USB-C6, K1 TACT_6x6_SMD, K10 TACT_6x6_SMD, K11 TACT_6x6_SMD, K12 TACT_6x6_SMD, K13 TACT_6x6_SMD, K14 TACT_6x6_SMD, K15 TACT_6x6_SMD, K16 TACT_6x6_SMD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

Commit message: Projektowanie płytki
Connections:
- net 3V3: now also DISP1.2 (Pin_2); no longer DISP1.1 (Pin_1)
- net GND: now also DISP1.1 (Pin_1); no longer DISP1.2 (Pin_2)
- net SCL: now also DISP1.3 (Pin_3); no longer DISP1.5 (Pin_5)
Changed lines of the file:
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@@
 	(wire
 		(pts
-			(xy 209.55 60.96) (xy 217.17 60.96)
+			(xy 210.82 63.5) (xy 217.17 63.5)
 		)
 		(stroke
@@
 	(wire
 		(pts
-			(xy 210.82 55.88) (xy 217.17 55.88)
+			(xy 210.82 68.58) (xy 217.17 68.58)
 		)
 		(stroke
@@
 	(wire
 		(pts
-			(xy 209.55 63.5) (xy 217.17 63.5)
+			(xy 210.82 60.96) (xy 217.17 60.96)
 		)
 		(stroke
@@
 	(wire
 		(pts
-			(xy 210.82 66.04) (xy 217.17 66.04)
+			(xy 210.82 55.88) (xy 217.17 55.88)
 		)
 		(stroke
@@
 	(wire
 		(pts
-			(xy 210.82 68.58) (xy 217.17 68.58)
+			(xy 210.82 53.34) (xy 217.17 53.34)
 		)
 		(stroke
@@
 	(wire
 		(pts
-			(xy 210.82 53.34) (xy 217.17 53.34)
+			(xy 210.82 66.04) (xy 217.17 66.04)
 		)
 		(stroke
@@
 	)
 	(label "3V3"
-		(at 210.82 53.34 0)
+		(at 210.82 66.04 0)
 		(effects
 			(font
@@
 	)
 	(label "SCL"
-		(at 209.55 63.5 0)
+		(at 210.82 63.5 0)
 		(effects
 			(font
@@
 	)
 	(label "GND"
-		(at 210.82 55.88 0)
+		(at 210.82 68.58 0)
 		(effects
 			(font
@@
 	)
 	(label "SDA"
-		(at 209.55 60.96 0)
+		(at 210.82 60.96 0)
 		(effects
 			(font
@@
 	)
 	(label "3V3"
-		(at 210.82 68.58 0)
+		(at 210.82 53.34 0)
 		(effects
 			(font
@@
 	)
 	(label "GND"
-		(at 210.82 66.04 0)
+		(at 210.82 55.88 0)
 		(effects
 			(font
@@
 		(lib_id "Connector_Generic:Conn_01x07")
 		(at 222.25 60.96 0)
+		(mirror x)
 		(unit 1)
 		(exclude_from_sim no)
@@
 		(dnp no)
 		(property "Reference" "DISP1"
-			(at 222.25 50.8 0)
+			(at 222.25 71.12 0)
 			(effects
 				(font
@@
 		)
 		(property "Value" "OLED"
-			(at 222.25 71.12 0)
+			(at 222.25 50.8 0)
 			(effects
 				(font
