File: Nostalgia.kicad_pcb (KiCad board)
At the start: 2 copper layers, 72 x 122 mm, 59 parts, among them J10 490107670612, J20 USB-C6, K1 TACT_6x3_SMD, K10 TACT_6x3_SMD, K11 TACT_6x3_SMD, K12 TACT_6x3_SMD, K13 TACT_6x6_SMD, K14 TACT_6x6_SMD, K15 TACT_6x6_SMD, K16 TACT_6x6_SMD, K2 TACT_6x3_SMD, K3 TACT_6x3_SMD, K4 TACT_6x3_SMD, K5 TACT_6x3_SMD, K6 TACT_6x3_SMD, K7 TACT_6x3_SMD, K8 TACT_6x3_SMD, K9 TACT_6x3_SMD, U1 TP4056, U2 TPS63000, U40 ESP32-S3-WROOM-1-N16R8, U5 TPS613222ADBV

Commit message: WIP
Parts:
- removed C4, C42, C44, C5: 10u, _custom:C_0603
- removed C40, C41, C43: 100n, _custom:C_0603
- removed the DISP1 at (114.5, -54.3)
- removed L4: 4.7uH, _custom:DJNR3015
- removed R40: 10k, _custom:R_0603
- removed R7: 1M, _custom:R_0603
- removed TP3: 5V, _custom:Testpoint_2.00mm
- removed U5: TPS613222ADBV, _custom:SOT23-5
- added C11: 100n, _custom:C_0805, B.Cu at (49.0, -107.7)
- added C12: 10u, _custom:C_0805, B.Cu at (51.0, -107.7)
- added C13: 100n, _custom:C_0805, B.Cu at (53.0, -107.7)
- added C14: 10u, _custom:C_0805, B.Cu at (53.0, -104.4)
- added PMOD1: Conn_02x06_Top_Bottom, _custom:PMOD, F.Cu at (10.0, -142.5)
- added PMOD2: Conn_02x06_Top_Bottom, _custom:PMOD, F.Cu at (62.1, -124.3)
- added R10: 10k, _custom:R_0805, B.Cu at (51.0, -104.4)
- C1, C2, C3, C6, C7, C8: footprint _custom:C_0603 -> _custom:C_0805; moved to B.Cu
- C10: value 10u -> 1u; footprint _custom:C_0603 -> _custom:C_0805; moved to B.Cu
- D1, D2, L1, TP1, TP4, U1, U2: moved to B.Cu
- DISP1: renamed from DISP2; footprint _custom:OLED_2.42inch_board_2 -> _custom:OLED_2.42inch_board_3
- K1, K10, K11, K12, K2, K3, K4, K5, K6, K7, K8, K9: value TACT_6x3_SMD -> TACT_6x6_SMD
- R1, R2, R20, R21, R3, R4, R5, R6: footprint _custom:R_0603 -> _custom:R_0805; moved to B.Cu
- moved C10 132.3 mm to (49.0, -104.4), turned to -90 degrees
- moved U1 100.6 mm to (57.5, -88.8), turned to 180 degrees
- moved J10 53.2 mm to (67.8, -106.5), turned to -90 degrees
- moved C3 25.6 mm to (86.1, 9.25), turned to 180 degrees
- moved C6 25.6 mm to (86.1, 11.2), turned to 180 degrees
- moved C7 25.6 mm to (86.1, 13.2), turned to 180 degrees
- moved C8 25.6 mm to (86.1, 15.1), turned to 180 degrees
- moved R4 25.6 mm to (86.1, 17.1), turned to 180 degrees
- moved R5 25.6 mm to (86.1, 19.0), turned to 180 degrees
- moved R6 25.6 mm to (86.1, 20.9), turned to 180 degrees
- moved C2 20.9 mm to (128.5, -7.67), turned to 180 degrees
- moved U10 20.0 mm to (36.0, -115.2)
- moved D1 19.9 mm to (128.0, -12.2), turned to 180 degrees
- moved D2 19.9 mm to (128.0, -9.85), turned to 180 degrees
- moved C1 10.4 mm to (112.9, -12.3), turned to 180 degrees
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- renumbered U40 to U10
Connections:
- C10 pad 1: VBAT -> /Reset
- K13 pad 1: /Col3 -> GND
- K13 pad 2: /Row2 -> /ButtonLeft
- K14 pad 1: /Col3 -> GND
- K14 pad 2: /Row0 -> /ButtonUp
- K15 pad 1: /Col3 -> GND
- K15 pad 2: /Row1 -> /ButtonDown
- K16 pad 1: /Col3 -> GND
- K16 pad 2: /Row3 -> /ButtonRigth
Routing:
- net /Col2: track 0.00 -> 65.0 mm, vias 0 -> 4
- net /Col1: track 0.00 -> 65.0 mm, vias 0 -> 4
- net /Col0: track 0.00 -> 65.0 mm, vias 0 -> 4
- net /Row0: track 0.00 -> 64.0 mm, vias 0 -> 4
- net /Row3: track 0.00 -> 63.8 mm, vias 0 -> 4
- net /Row2: track 0.00 -> 63.8 mm, vias 0 -> 4
- net /Row1: track 0.00 -> 63.8 mm, vias 0 -> 4
- net GND: vias 0 -> 125
- added copper zone on B.Cu, net GND
- added copper zone on F.Cu, net GND

Commit message: WIP
Parts:
- moved J10 34.5 mm to (36.0, -93.0), turned to 0 degrees
- moved PMOD1 32.2 mm to (13.5, -110.5), turned to -90 degrees
- moved PMOD2 14.3 mm to (58.5, -110.5)
- moved DISP1 0.25 mm to (36.0, -100.0)
- turned K13 to 180 degrees
- turned K15 to 180 degrees
- turned K16 to 180 degrees
Other:
- board text added: "122"
- board text added: "72"
- board text removed: "102"

Commit message: Schemat prawie gotowy
Parts:
- added C22: 100n, _custom:C_0805, B.Cu at (16.4, 9.93)
- added C40: 100n, _custom:C_0805, B.Cu at (16.4, 12.3)
- added C41: 10u, _custom:C_0805, B.Cu at (16.4, 14.7)
- added R25: xxx, _custom:R_0805, B.Cu at (16.4, 17.1)
- added R26: xxx, _custom:R_0805, B.Cu at (16.4, 19.5)
- L30: renamed from L1; footprint _custom:DJNR3015 -> _custom:DJNR5050
- moved C20 106.7 mm to (61.2, -90.5), turned to -90 degrees
- moved R21 104.9 mm to (65.5, -81.2), turned to 90 degrees
- moved R20 102.4 mm to (63.5, -81.2), turned to 90 degrees
- moved TP1 51.9 mm to (12.8, 10.5)
- moved TP4 48.9 mm to (12.8, 14.1)
- moved C12 11.6 mm to (48.8, -119.0), turned to 0 degrees
- moved C13 10.3 mm to (48.8, -117.0), turned to 0 degrees
- moved C14 9.59 mm to (48.8, -113.0), turned to 0 degrees
- moved C11 7.35 mm to (48.8, -115.0), turned to 0 degrees
- moved C10 6.60 mm to (48.8, -111.0), turned to 0 degrees
- moved R10 5.12 mm to (48.8, -109.0), turned to 0 degrees
- renumbered C2 to C20, C1 to C21, C3 to C30, C7 to C31, C6 to C32, C8 to C33, R1 to R22, R2 to R23, R3 to R24, R6 to R30, R4 to R31, R5 to R32, U1 to U20, U2 to U30
Connections:
- DISP1 pad 1: unconnected-(DISP1-Pin_1-Pad1) -> 3V3
- DISP1 pad 2: unconnected-(DISP1-Pin_2-Pad2) -> GND
- DISP1 pad 4: unconnected-(DISP1-Pin_4-Pad4) -> /SDA
- DISP1 pad 5: unconnected-(DISP1-Pin_5-Pad5) -> /SCL
- DISP1 pad 6: unconnected-(DISP1-Pin_6-Pad6) -> GND
- DISP1 pad 7: unconnected-(DISP1-Pin_7-Pad7) -> 3V3
- PMOD1 pad 1: unconnected-(PMOD1-Pin_1-Pad1) -> /GPIO10
- PMOD1 pad 10: unconnected-(PMOD1-Pin_10-Pad10) -> /GPIO8
- PMOD1 pad 2: unconnected-(PMOD1-Pin_2-Pad2) -> /GPIO11
- PMOD1 pad 3: unconnected-(PMOD1-Pin_3-Pad3) -> /GPIO13
- PMOD1 pad 4: unconnected-(PMOD1-Pin_4-Pad4) -> /GPIO12
- PMOD1 pad 7: unconnected-(PMOD1-Pin_7-Pad7) -> /GPIO15
- PMOD1 pad 8: unconnected-(PMOD1-Pin_8-Pad8) -> /GPIO14
- PMOD1 pad 9: unconnected-(PMOD1-Pin_9-Pad9) -> /GPIO9
- PMOD2 pad 1: unconnected-(PMOD2-Pin_1-Pad1) -> /GPIO39
- PMOD2 pad 10: unconnected-(PMOD2-Pin_10-Pad10) -> /GPIO48
- PMOD2 pad 2: unconnected-(PMOD2-Pin_2-Pad2) -> /GPIO40
- PMOD2 pad 3: unconnected-(PMOD2-Pin_3-Pad3) -> /GPIO41
- PMOD2 pad 4: unconnected-(PMOD2-Pin_4-Pad4) -> /GPIO42
- PMOD2 pad 7: unconnected-(PMOD2-Pin_7-Pad7) -> /GPIO45
- PMOD2 pad 8: unconnected-(PMOD2-Pin_8-Pad8) -> /GPIO46
- PMOD2 pad 9: unconnected-(PMOD2-Pin_9-Pad9) -> /GPIO47
- U10 pad 10: unconnected-(U10-Tx1/IO17-Pad10) -> /Row1
- U10 pad 11: unconnected-(U10-Rx1/IO18-Pad11) -> /Row2
- U10 pad 12: unconnected-(U10-IO8-Pad12) -> /GPIO8
- U10 pad 13: unconnected-(U10-D-/IO19-Pad13) -> /Row3
- U10 pad 14: unconnected-(U10-D+/IO20-Pad14) -> /Col0
- U10 pad 15: unconnected-(U10-JTAG/IO3-Pad15) -> /SDA
- U10 pad 16: unconnected-(U10-Log/IO46-Pad16) -> /GPIO46
- U10 pad 17: unconnected-(U10-IO9-Pad17) -> /GPIO9
- U10 pad 18: unconnected-(U10-IO10-Pad18) -> /GPIO10
- U10 pad 19: unconnected-(U10-IO11-Pad19) -> /GPIO11
- U10 pad 20: unconnected-(U10-IO12-Pad20) -> /GPIO12
- U10 pad 21: unconnected-(U10-IO13-Pad21) -> /GPIO13
- U10 pad 22: unconnected-(U10-IO14-Pad22) -> /GPIO14
- U10 pad 23: unconnected-(U10-IO21-Pad23) -> /Col1
- U10 pad 24: unconnected-(U10-IO47-Pad24) -> /GPIO47
- U10 pad 25: unconnected-(U10-IO48-Pad25) -> /GPIO48
- U10 pad 26: unconnected-(U10-MemVolt/IO45-Pad26) -> /GPIO45
- U10 pad 31: unconnected-(U10-IO38-Pad31) -> /Col2
- U10 pad 32: unconnected-(U10-MTCK/IO39-Pad32) -> /GPIO39
- U10 pad 33: unconnected-(U10-MTDO/IO40-Pad33) -> /GPIO40
- U10 pad 34: unconnected-(U10-MTDI/IO41-Pad34) -> /GPIO41
- U10 pad 35: unconnected-(U10-MTMS/IO42-Pad35) -> /GPIO42
- U10 pad 38: unconnected-(U10-IO2-Pad38) -> /SCL
- U10 pad 39: unconnected-(U10-IO1-Pad39) -> /ADC-Bat
- U10 pad 4: unconnected-(U10-IO4-Pad4) -> /ButtonUp
- U10 pad 5: unconnected-(U10-IO5-Pad5) -> /ButtonDown
- U10 pad 6: unconnected-(U10-IO6-Pad6) -> /ButtonLeft
- U10 pad 7: unconnected-(U10-IO7-Pad7) -> /ButtonRigth
- U10 pad 8: unconnected-(U10-XTAL/IO15-Pad8) -> /GPIO15
- U10 pad 9: unconnected-(U10-XTAL/IO16-Pad9) -> /Row0
Other:
- board text added: "3V3"

Commit message: WIP
Parts:
- added REF**: SW_NKK_BB15AH, Button_Switch_THT:SW_NKK_BB15AH, F.Cu at (78.7, -88.4)
- added REF**: SW_Push_1P2T_Vertical_E-Switch_800UDP8P1A1M6, Button_Switch_THT:SW_Push_1P2T_Vertical_E-Switch_800UDP8P1A1M6, F.Cu at (92.0, -104.2)
- moved D2 106.7 mm to (70.5, -99.8), turned to -90 degrees
- moved D1 101.8 mm to (70.5, -96.2), turned to -90 degrees
Other:
- board text added: "10"
- board text added: "11"
- board text added: "12"
- board text added: "13"
- board text added: "14"
- board text added: "15"
- board text added: "39"
- board text added: "40"
- board text added: "41"
- board text added: "42"
- board text added: "45"
- board text added: "46"
- board text added: "47"
- board text added: "48"
- board text added: "8"
- board text added: "9"
- board text added: "GND"

Commit message: Włącznik zasilania
Parts:
- removed REF**: SW_NKK_BB15AH, Button_Switch_THT:SW_NKK_BB15AH
- removed REF**: SW_Push_1P2T_Vertical_E-Switch_800UDP8P1A1M6, Button_Switch_THT:SW_Push_1P2T_Vertical_E-Switch_800UDP8P1A1M6
- added K17: YUEN_FUNG_ST-0-102-C03-N003-RS, _custom:YUEN_FUNG_ST-0-102-C03-N003-RS, F.Cu at (59.8, -99.0)
- moved D2 1.77 mm to (70.8, -101.5)
- moved D1 0.35 mm to (70.8, -96.5)
Connections:
- BAT1 pad 1: VBAT -> Net-(BAT1-+)
- BAT2 pad 1: VBAT -> Net-(BAT1-+)
- BAT3 pad 1: VBAT -> Net-(BAT1-+)
- C21 pad 1: VBAT -> Net-(BAT1-+)
- R25 pad 2: VBAT -> Net-(BAT1-+)
- U20 pad 5: VBAT -> Net-(BAT1-+)

Commit message: Projektowanie płytki
Parts:
- C10, C11, C12, C13, C14, C20, C21, C22, C30, C31, C32, C33, C40, C41, D1, D2, J20, L30, R10, R20, R21, R22, R23, R24, R25, R26, R30, R31, R32, U20, U30: moved to F.Cu
- moved R32 120.6 mm to (45.5, -94.5), turned to -90 degrees
- moved R30 117.2 mm to (51.5, -91.0), turned to -90 degrees
- moved R31 115.4 mm to (45.5, -91.0), turned to -90 degrees
- moved U30 113.3 mm to (48.5, -92.8), turned to 90 degrees
- moved C31 113.1 mm to (51.5, -94.5), turned to 90 degrees
- moved C33 110.1 mm to (43.8, -86.5), turned to -90 degrees
- moved C41 108.8 mm to (7.50, -93.8), turned to -90 degrees
- moved C32 107.3 mm to (41.8, -86.5), turned to -90 degrees
- moved C40 106.6 mm to (5.50, -93.8), turned to -90 degrees
- moved C30 105.4 mm to (53.5, -91.0), turned to 90 degrees
- moved R26 102.5 mm to (15.2, -83.0), turned to 90 degrees
- moved L30 101.8 mm to (48.5, -86.5), turned to 0 degrees
- moved R23 100.3 mm to (66.5, -97.2), turned to 0 degrees
- moved R25 100.2 mm to (13.0, -83.0), turned to -90 degrees
- moved R22 96.8 mm to (66.5, -95.2), turned to 0 degrees
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Connections:
- DISP1 pad 1: 3V3 -> GND
- DISP1 pad 2: GND -> 3V3
- DISP1 pad 3: unconnected-(DISP1-Pin_3-Pad3) -> /SCL
- DISP1 pad 5: /SCL -> unconnected-(DISP1-Pin_5-Pad5)
Routing:
- net GND: track 0.00 -> 93.2 mm
- net Net-(BAT1-+): track 0.00 -> 83.0 mm, vias 0 -> 1
- net VUSB: track 0.00 -> 42.5 mm
- net VBAT: track 0.00 -> 14.8 mm
- net Net-(J20-CC2): track 0.00 -> 10.6 mm
- net Net-(J20-CC1): track 0.00 -> 10.5 mm
- net Net-(U20-~{CHRG}): track 0.00 -> 10.3 mm
- net /ButtonUp: track 0.00 -> 8.50 mm
- net /ButtonRigth: track 0.00 -> 8.50 mm
- net /ButtonLeft: track 0.00 -> 8.50 mm
- net /ButtonDown: track 0.00 -> 8.50 mm
- net Net-(U20-~{STDBY}): track 0.00 -> 8.18 mm
- net Net-(U30-EN): track 0.00 -> 8.04 mm
- net Net-(U30-L2): track 0.00 -> 5.48 mm
- net Net-(U30-L1): track 0.00 -> 5.48 mm
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